Commit message: feat: align gripper range and add external simulation collection API

File: assets/mujoco/kinematics.urdf (robot description, URDF)
Before this commit: robot piper, 11 links, 10 joints
Joints:
- joint joint7: limit lower=0 upper=0.035 effort=10 velocity=0.1 -> lower=0 upper=0.0475 effort=10 velocity=0.1
- joint joint8: limit lower=0 upper=0.035 effort=10 velocity=0.1 -> lower=0 upper=0.0475 effort=10 velocity=0.1
